File: Terasaki_V.1/Schematic/Terasaki_V.1.kicad_sch (KiCad schematic)
At the start: 61 parts, among them J3 52610-1572, J4 1053091202, J5 1053091203, J6 1053091202, SW1 K2-1808SN-A4SW, SW2 K2-1808SN-A4SW, SW3 2MS1T2B2M6QES, U1 ESP32-S3-MINI-1-N4R2, U2 AP2114H-3.3TRG1, U3 TPD2E001DRYR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

Commit message: Add files via upload
Parts:
- removed C17, C7, C8: 10uF, easyeda2kicad:C0805, symbol easyeda2kicad:CL21A106KOQNNNE
- removed C18, C24, C4: 100nF, easyeda2kicad:C0603, symbol easyeda2kicad:GRM188R71C104KA01D
- removed U2: AP2114H-3.3TRG1, easyeda2kicad:SOT-223_L6.7-W3.5-P2.30-BR, symbol easyeda2kicad:AP2114H-3.3TRG1
- added C17, C18: 10uF, easyeda2kicad:C0805, symbol easyeda2kicad:CL21B106KPQNNNE
- added C24: 10uF, easyeda2kicad:C0805, symbol easyeda2kicad:CL21A106KOQNNNE
- added C27, C34, C35: 100nF, easyeda2kicad:C0603, symbol easyeda2kicad:GRM188R71C104KA01D
- added C37, C38, C39: 1uF, easyeda2kicad:C0603, symbol easyeda2kicad:CL10B105KP8NNNC
- added H1: A2541WV-5P, easyeda2kicad:HDR-TH_5P-P2.54-V-M, symbol easyeda2kicad:A2541WV-5P
- added L2: BLM18AG601SN1D, easyeda2kicad:L0603, symbol easyeda2kicad:BLM18AG601SN1D
- added R7: 2.2Ω, easyeda2kicad:R0402, symbol easyeda2kicad:RC0402FR-072R2L
- added U5: ADM7150ARDZ-3.3-R7, easyeda2kicad:SOIC-8_L4.9-W3.9-P1.27-LS6.0-BL-EP3.1, symbol easyeda2kicad:ADM7150ARDZ-3.3-R7
Connections:
- net +3V3: now also C17.2, C35.2, L2.1, U5.2 (VOUT); no longer U4.30 (AVDD), U4.41 (AVDD)
- net +5V: now also R6.1
- net GND: now also C17.1, C18.1, C24.1, C27.1, C34.1, C35.1, C37.2, C38.2, C39.2, U5.4 (GND), U5.9 (EP); no longer R6.1
- net VCC: now also C18.2, U5.7 (EN), U5.8 (VIN)
- net A2: now reaches U6.15 (A2)
- net A2: now also U1.14 (IO10), U7.15 (A2), U8.15 (A2)
- net AIN3: now reaches U4.36 (AIN3/BUF_VREF1V8)
- net AIN3: now also H1.2
- net AIN2: now reaches U4.37 (AIN2)
- net AIN2: now also H1.3
- net AIN1: now reaches U4.38 (AIN1)
- net AIN1: now also H1.4
- net AIN0: now reaches U4.39 (AIN0)
- net AIN0: now also H1.5
- net AIN4: now reaches U4.40 (AIN4/LPF0)
- net AIN4: now also H1.1
- new net: L2.2, R7.1
- new net: C38.1, U5.1 (VREG)
- new net: C37.1, U5.3 (BYP)
- new net: C39.1, U5.5 (REF_SENSE), U5.6 (REF)
- new net AVDD: C24.2, C27.2, C34.2, R7.2, U4.30 (AVDD), U4.41 (AVDD)
- no-connect marks 78 -> 69
Other:
- note added: "Analog In"
- moved on the sheet: C10, C16, C28, C29, C30, C31, C32, C33, D2, D3, J3, LED1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
